File: templates/default-4layer/default-4layer.kicad_pcb (KiCad board)
At the start: 4 copper layers, 0 parts

Commit message: Starting to update templates.
Other:
- copper layers 4 -> 2
Changed lines of the file:
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@@
   (layers
     (0 F.Cu signal)
-    (1 In1.Cu signal)
-    (2 In2.Cu signal)
     (31 B.Cu signal)
+    (33 F.Adhes user)
     (34 B.Paste user)
     (35 F.Paste user)
@@
     (38 B.Mask user)
     (39 F.Mask user)
+    (40 Dwgs.User user)
     (44 Edge.Cuts user)
-    (46 B.CrtYd user)
-    (47 F.CrtYd user)
     (48 B.Fab user)
     (49 F.Fab user)
@@
     (uvia_drill 0.3302)
   )
-  (gr_circle (center 117.348 76.962) (end 118.618 76.962) (layer Dwgs.User) (width 0.15))
-  (gr_line (start 114.427 78.994) (end 114.427 74.93) (angle 90) (layer Dwgs.User) (width 0.15))
-  (gr_line (start 120.269 78.994) (end 114.427 78.994) (angle 90) (layer Dwgs.User) (width 0.15))
-  (gr_line (start 120.269 74.93) (end 120.269 78.994) (angle 90) (layer Dwgs.User) (width 0.15))
-  (gr_line (start 114.427 74.93) (end 120.269 74.93) (angle 90) (layer Dwgs.User) (width 0.15))
-  (gr_line (start 120.523 93.98) (end 104.648 93.98) (angle 90) (layer Dwgs.User) (width 0.15))
-  (gr_line (start 173.355 102.235) (end 173.355 94.615) (angle 90) (layer Dwgs.User) (width 0.15))
-  (gr_line (start 178.435 102.235) (end 173.355 102.235) (angle 90) (layer Dwgs.User) (width 0.15))
-  (gr_line (start 178.435 94.615) (end 178.435 102.235) (angle 90) (layer Dwgs.User) (width 0.15))
-  (gr_line (start 173.355 94.615) (end 178.435 94.615) (angle 90) (layer Dwgs.User) (width 0.15))
-  (gr_line (start 109.093 123.19) (end 109.093 114.3) (angle 90) (layer Dwgs.User) (width 0.15))
-  (gr_line (start 122.428 123.19) (end 109.093 123.19) (angle 90) (layer Dwgs.User) (width 0.15))
-  (gr_line (start 122.428 114.3) (end 122.428 123.19) (angle 90) (layer Dwgs.User) (width 0.15))
-  (gr_line (start 109.093 114.3) (end 122.428 114.3) (angle 90) (layer Dwgs.User) (width 0.15))
-  (gr_line (start 104.648 93.98) (end 104.648 82.55) (angle 90) (layer Dwgs.User) (width 0.15))
-  (gr_line (start 120.523 82.55) (end 120.523 93.98) (angle 90) (layer Dwgs.User) (width 0.15))
-  (gr_line (start 104.648 82.55) (end 120.523 82.55) (angle 90) (layer Dwgs.User) (width 0.15))
 )
